File: uLements_v2.5.sch (EAGLE design)
At the start: 189 parts, among them IC1 LM4040B10, IC10 STM32F405RGT6, IC11 4051PW, IC12 WM8731, IC13 MCP6004-I_ST, IC14 LME49720, IC2 LM1117-3.3, IC3 4051PW, IC4 LM1117-3.3, IC5 4051PW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

Commit message: uLements files
Other:
- note added: "Codex-Modulex"
- note added: "Original design by: Olivier Gillet of Mutable Instruments"
- note added: "info@codex-modulex.com"
- note removed: "Olivier Gillet"
- note removed: "ol.gillet@gmail.com"
